File: Robot.kicad_sch (KiCad schematic)
At the start: 0 parts

Commit message: [PCB][SCH] Add temporary (for CI) moddifs
Other:
- note added: "TEMPORARY"
Changed lines of the file:
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@@
 (kicad_sch (version 20220404) (generator eeschema)
   (paper "A4")
-  (symbol_instances)
+  (text "TEMPORARY" (at 15.24 16.51 0)
+    (effects (font (size 1.27 1.27)) (justify left bottom))
+  )
+  (sheet_instances
+    (path "/" (page "1"))
+  )
 )
